File: Kicad/reaction_game.kicad_pcb (KiCad board)
At the start: 2 copper layers, 95 x 67.5 mm, 12 parts, among them SW1 Player 1, SW2 Player 2, U1 RaspberryPico

Commit message: 3D models, placement
Parts:
- removed H5: MountingHole_NPTH, MM_Various:MountingHole_3.2mm_M3_Pad_NPTH
- moved R2 49.4 mm to (114.5, 74.5), turned to 180 degrees
- moved H3 45.5 mm to (103.5, 96.5)
- moved R1 35.6 mm to (147.5, 60.0), turned to -90 degrees
- moved R3 33.9 mm to (183.0, 75.0), turned to 180 degrees

Commit message: Finished routing
Connections:
- U1 pad 1: /Button_1 -> /LED_1
- U1 pad 2: /LED_1 -> /Button_1
Routing:
- net +3V3: track 0.00 -> 156.4 mm
- net /Button_2: track 0.00 -> 82.1 mm
- net /LED_2: track 0.00 -> 68.6 mm
- net /Button_1: track 0.00 -> 51.1 mm
- net /LED_1: track 0.00 -> 27.5 mm
- net /Game_LED: track 0.00 -> 13.0 mm
- net Net-(SW1-A): track 0.00 -> 5.44 mm
- net Net-(SW2-A): track 0.00 -> 4.92 mm
- net Net-(D1-A): track 0.00 -> 4.68 mm
- added copper zone on B.Cu, net GND
- added copper zone on F.Cu, net GND
Other:
- board text added: "2025 MM & SM"
- board text added: "Reaction Game"

Commit message: Silkscreen
Routing:
- net +3V3: track 156.4 -> 158.9 mm
- net GND: vias 0 -> 36
